File: pcbs/main_pcb.kicad_pcb (KiCad board)
At the start: 2 copper layers, 139.3 x 147.8 mm, 60 parts

Commit message: fix
Parts:
- moved TRRS1 3.53 mm to (267.4, 122.1)
- moved D7 3.53 mm to (159.7, 121.1)
- moved B1 3.53 mm to (249.9, 120.1)
- moved S2 3.53 mm to (140.7, 135.2)
- moved S13 3.53 mm to (197.8, 138.2)
- moved D16 3.53 mm to (197.8, 86.1)
- moved D11 3.53 mm to (178.8, 113.1)
- moved S15 3.53 mm to (197.8, 100.1)
- moved D20 3.53 mm to (216.9, 94.1)
- moved S9 3.53 mm to (178.8, 146.2)
- moved D5 3.53 mm to (159.7, 159.2)
- moved D1 3.53 mm to (140.7, 159.2)
- moved S3 3.53 mm to (140.7, 116.1)
- moved _1 3.53 mm to (150.2, 106.6)
- moved D25 3.53 mm to (232.4, 182.7)
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Connections:
- S13 pad 1: P07 -> P7
- S14 pad 1: P07 -> P7
- S15 pad 1: P07 -> P7
- S16 pad 1: P07 -> P7
- S17 pad 1: P08 -> P8
- S18 pad 1: P08 -> P8
- S19 pad 1: P08 -> P8
- S20 pad 1: P08 -> P8
- S21 pad 1: P09 -> P9
- S22 pad 1: P09 -> P9
- S23 pad 1: P09 -> P9
- S24 pad 1: P09 -> P9
- S25 pad 1: P08 -> P8
- S26 pad 1: P09 -> P9
Routing:
- net P9: track 0.00 -> 230.1 mm, vias 0 -> 5
- net P8: track 0.00 -> 208.2 mm, vias 0 -> 5
- net P14: track 0.00 -> 156.3 mm, vias 0 -> 4
- net P7: track 0.00 -> 151.7 mm, vias 0 -> 4
- net P10: track 0.00 -> 151.6 mm, vias 0 -> 4
- net P21: track 23.8 -> 173.9 mm
- net P16: track 0.00 -> 132.9 mm, vias 0 -> 4
- net inner_num: track 16.5 -> 33.3 mm, vias 0 -> 1
- net inner_bottom: track 16.5 -> 33.1 mm, vias 0 -> 1
- net aditional_bottom: track 16.6 -> 32.9 mm, vias 0 -> 1
- net index_bottom: track 16.5 -> 32.9 mm, vias 0 -> 1
- net middle_bottom: track 16.6 -> 32.9 mm, vias 0 -> 1
- net middle_home: track 16.6 -> 32.8 mm, vias 0 -> 1
- net aditional_home: track 16.4 -> 32.7 mm, vias 0 -> 1
- net index_home: track 16.5 -> 32.8 mm, vias 0 -> 1
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Other:
- outline, holes or cut-outs redrawn

Commit message: att
Parts:
- MCU1: value (none) -> nice!nano_v2; footprint ProMicro -> nice!nano_v2
- moved MCU1 10.3 mm to (266.2, 90.6), turned to 0 degrees
- moved TRRS1 10.2 mm to (276.8, 117.9)
- moved S2 10.2 mm to (150.0, 130.9)
- moved D7 10.2 mm to (169.1, 116.9)
- moved S13 10.2 mm to (207.2, 134.0)
- moved _2 10.2 mm to (159.5, 140.5)
- moved D20 10.2 mm to (226.2, 89.8)
- moved S15 10.2 mm to (207.2, 95.9)
- moved D11 10.2 mm to (188.1, 108.9)
- moved D23 10.2 mm to (245.2, 116.9)
- moved S21 10.2 mm to (245.2, 150.0)
- moved D1 10.2 mm to (150.0, 155.0)
- moved B1 10.2 mm to (259.2, 115.9)
- moved D15 10.2 mm to (207.2, 100.9)
- moved D9 10.2 mm to (188.1, 147.0)
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Routing:
- net P9: track 230.1 -> 9.13 mm, vias 5 -> 0
- net P8: track 208.2 -> 9.13 mm, vias 5 -> 0
- net P21: track 173.9 -> 9.26 mm
- net P14: track 156.3 -> 9.20 mm, vias 4 -> 0
- net P10: track 151.6 -> 9.13 mm, vias 4 -> 0
- net P7: track 151.7 -> 9.74 mm, vias 4 -> 0
- net P16: track 132.9 -> 9.20 mm, vias 4 -> 0
- net inner_num: track 33.3 -> 0.00 mm, vias 1 -> 0
- net inner_bottom: track 33.1 -> 0.00 mm, vias 1 -> 0
- net aditional_bottom: track 32.9 -> 0.00 mm, vias 1 -> 0
- net middle_bottom: track 32.9 -> 0.00 mm, vias 1 -> 0
- net inner_home: track 32.9 -> 0.00 mm, vias 1 -> 0
- net pinky_top: track 32.9 -> 0.00 mm, vias 1 -> 0
- net index_bottom: track 32.9 -> 0.00 mm, vias 1 -> 0
- net middle_home: track 32.8 -> 0.00 mm, vias 1 -> 0
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Other:
- outline, holes or cut-outs redrawn

Commit message: att
Routing:
- net P7: track 9.74 -> 9.13 mm

Commit message: gerbers
Routing:
- net P14: track 9.20 -> 280.8 mm, vias 0 -> 2
- net P16: track 9.20 -> 278.2 mm, vias 0 -> 6
- net P8: track 9.13 -> 241.4 mm, vias 0 -> 7
- net P18: track 9.13 -> 228.1 mm, vias 0 -> 1
- net P9: track 9.13 -> 226.6 mm, vias 0 -> 4
- net P10: track 9.13 -> 225.7 mm, vias 0 -> 4
- net P19: track 9.13 -> 203.1 mm, vias 0 -> 1
- net P20: track 9.13 -> 199.8 mm, vias 0 -> 2
- net P7: track 9.13 -> 195.5 mm, vias 0 -> 4
- net P21: track 9.26 -> 170.9 mm, vias 0 -> 1
- net P15: track 9.26 -> 149.9 mm, vias 0 -> 1
- net GND: track 31.9 -> 93.0 mm, vias 0 -> 1
- net P0: track 9.13 -> 58.8 mm
- net RST: track 9.13 -> 50.5 mm
- net VCC: track 9.26 -> 46.7 mm
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